Commit message: refactor!: adopt the litearm_description joint and link naming
The arm description this stack builds against is `litearm_description`, whose URDF
names its joints `Joint1..Joint7`, its links `Link1..Link7` and its tool flange
`ee_frame_link`. The control block, the controller config, the joint-name parsing
and the tests still used the previous generation's lowercase `joint1..joint7`:

- `src/litearm_system.cpp`: `kPrefix` is `"Joint"` now -- the name is the mapping
  contract to the firmware axis, so this is the one line that makes the block bind
- `urdf/litearm.ros2_control.xacro`: the seven `<joint name="...">` entries
- `config/litearm_controllers.yaml`: the controller's joint lists
- `test/test_litearm_system.cpp`: the fixtures
- READMEs and docs

BREAKING CHANGE: the `<ros2_control>` block only binds a description whose joints
are named `Joint1..Joint7`.

File: litearm_ros2_control/urdf/litearm.ros2_control.xacro (robot description, xacro)
@@ -33,9 +33,9 @@
       <param name="reset_faults_on_configure">$(arg litearm_reset_faults_on_configure)</param>
     </hardware>
-    <!-- The joint names must be joint1..jointN, one per axis: the name is the
+    <!-- The joint names must be Joint1..jointN, one per axis: the name is the
          contract that maps a URDF joint to a firmware axis, so the order of the
          <joint> elements does not matter. N must equal the axis count the
          firmware reports (7 for the arm, 1 for the bench). -->
-    <joint name="joint1">
+    <joint name="Joint1">
       <command_interface name="position"/>
       <command_interface name="velocity"/>
@@ -54,5 +54,5 @@
       </xacro:if>
     </joint>
-    <joint name="joint2">
+    <joint name="Joint2">
       <command_interface name="position"/>
       <command_interface name="velocity"/>
@@ -67,5 +67,5 @@
       </xacro:if>
     </joint>
-    <joint name="joint3">
+    <joint name="Joint3">
       <command_interface name="position"/>
       <command_interface name="velocity"/>
@@ -80,5 +80,5 @@
       </xacro:if>
     </joint>
-    <joint name="joint4">
+    <joint name="Joint4">
       <command_interface name="position"/>
       <command_interface name="velocity"/>
@@ -93,5 +93,5 @@
       </xacro:if>
     </joint>
-    <joint name="joint5">
+    <joint name="Joint5">
       <command_interface name="position"/>
       <command_interface name="velocity"/>
@@ -106,5 +106,5 @@
       </xacro:if>
     </joint>
-    <joint name="joint6">
+    <joint name="Joint6">
       <command_interface name="position"/>
       <command_interface name="velocity"/>
@@ -119,5 +119,5 @@
       </xacro:if>
     </joint>
-    <joint name="joint7">
+    <joint name="Joint7">
       <command_interface name="position"/>
       <command_interface name="velocity"/>
